Commit message: 关节2重力补偿效果不好。其他两个可以
Co-authored-by: Copilot <copilot@github.com>

File: armurdf/armurdf_standard_motor/urdf/armurdf_standard_motor.urdf (robot description, URDF)
Before this commit: robot armurdf_standard_motor, 5 links, 4 joints
Joints:
- joint j1: origin xyz=0 0 0.07 rpy=1.5708 0 -1.5708 -> xyz=0 0 0.07 rpy=1.5708 0 1.57079265
